File: Solid State Relay Kit.sch (KiCad schematic (older format))
At the start: 11 parts, among them J1 Conn_01x03, J2 Conn_01x02, Q1 2N3904, U1 S108T02

Commit message: update,
Parts:
- D1, D2: footprint LEDs:LED_0805_HandSoldering -> LED_SMD:LED_0805_2012Metric_Castellated
- J1: footprint footprint-lib:Pin_Header_Straight_1x03_Pitch2.54mm -> Connector_PinHeader_2.54mm:PinHeader_1x03_P2.54mm_Vertical
- J2: footprint Connectors_Phoenix:PhoenixContact_MCV-G_02x5.08mm_Vertical -> w_conn_mpt:mpt_0,5%2f2-2,54
- Q1: footprint TO_SOT_Packages_SMD:TSOT-23_HandSoldering -> Package_TO_SOT_SMD:TSOT-23_HandSoldering
- R1, R2, R3, R4, R5: footprint Resistors_SMD:R_0805_HandSoldering -> Resistor_SMD:R_0805_2012Metric_Pad1.15x1.40mm_HandSolder
- U1: value S108T02 -> OMRON G3MB-202P; footprint Housings_SIP:SIP4_Sharp-SSR_Pitch7.62mm_Straight -> footprint-lib:OMRON-G3MB-202P
Changed lines of the file:
@@
 F 0 "J1" H 2720 2725 50  0000 C CNN
 F 1 "Conn_01x03" H 2720 2816 50  0000 C CNN
-F 2 "footprint-lib:Pin_Header_Straight_1x03_Pitch2.54mm" H 2800 3050 50  0001 C CNN
+F 2 "Connector_PinHeader_2.54mm:PinHeader_1x03_P2.54mm_Vertical" H 2800 3050 50  0001 C CNN
 F 3 "~" H 2800 3050 50  0001 C CNN
 	1    2800 3050
@@
 F 0 "R1" V 3443 2950 50  0000 C CNN
 F 1 "331" V 3534 2950 50  0000 C CNN
-F 2 "Resistors_SMD:R_0805_HandSoldering" V 3580 2950 50  0001 C CNN
+F 2 "Resistor_SMD:R_0805_2012Metric_Pad1.15x1.40mm_HandSolder" V 3580 2950 50  0001 C CNN
 F 3 "~" H 3650 2950 50  0001 C CNN
 	1    3650 2950
@@
 F 0 "R2" H 3970 3296 50  0000 L CNN
 F 1 "103" H 3970 3205 50  0000 L CNN
-F 2 "Resistors_SMD:R_0805_HandSoldering" V 3830 3250 50  0001 C CNN
+F 2 "Resistor_SMD:R_0805_2012Metric_Pad1.15x1.40mm_HandSolder" V 3830 3250 50  0001 C CNN
 F 3 "~" H 3900 3250 50  0001 C CNN
 	1    3900 3250
@@
 F 0 "R3" H 4270 2246 50  0000 L CNN
 F 1 "331" H 4270 2155 50  0000 L CNN
-F 2 "Resistors_SMD:R_0805_HandSoldering" V 4130 2200 50  0001 C CNN
+F 2 "Resistor_SMD:R_0805_2012Metric_Pad1.15x1.40mm_HandSolder" V 4130 2200 50  0001 C CNN
 F 3 "~" H 4200 2200 50  0001 C CNN
 	1    4200 2200
@@
 F 0 "D1" V 4238 1483 50  0000 R CNN
 F 1 "LED" V 4147 1483 50  0000 R CNN
-F 2 "LEDs:LED_0805_HandSoldering" H 4200 1600 50  0001 C CNN
+F 2 "LED_SMD:LED_0805_2012Metric_Castellated" H 4200 1600 50  0001 C CNN
 F 3 "~" H 4200 1600 50  0001 C CNN
 	1    4200 1600
@@
 F 0 "Q1" H 4641 2996 50  0000 L CNN
 F 1 "2N3904" H 4641 2905 50  0000 L CNN
-F 2 "TO_SOT_Packages_SMD:TSOT-23_HandSoldering" H 4650 2875 50  0001 L CIN
+F 2 "Package_TO_SOT_SMD:TSOT-23_HandSoldering" H 4650 2875 50  0001 L CIN
 F 3 "" H 4450 2950 50  0001 L CNN
 	1    4450 2950
@@
 P 5300 1850
 F 0 "U1" H 5300 2175 50  0000 C CNN
-F 1 "S108T02" H 5300 2084 50  0000 C CNN
-F 2 "Housings_SIP:SIP4_Sharp-SSR_Pitch7.62mm_Straight" H 5100 1650 50  0001 L CIN
-F 3 "http://cdn.sparkfun.com/datasheets/Components/General%20IC/S108,208T02%20Series.pdf" H 5265 1850 50  0001 L CNN
+F 1 "OMRON G3MB-202P" H 5300 2084 50  0000 C CNN
+F 2 "footprint-lib:OMRON-G3MB-202P" H 5100 1650 50  0001 L CIN
+F 3 "https://www.openhacks.com/uploadsproductos/g3mb-ssr-datasheet.pdf" H 5265 1850 50  0001 L CNN
 	1    5300 1850
 	1    0    0    -1
@@
 F 0 "J2" H 6719 1575 50  0000 C CNN
 F 1 "Conn_01x02" H 6719 1666 50  0000 C CNN
-F 2 "Connectors_Phoenix:PhoenixContact_MCV-G_02x5.08mm_Vertical" H 6800 1900 50  0001 C CNN
+F 2 "w_conn_mpt:mpt_0,5%2f2-2,54" H 6800 1900 50  0001 C CNN
 F 3 "~" H 6800 1900 50  0001 C CNN
 	1    6800 1900
@@
 F 0 "R4" H 4620 1596 50  0000 L CNN
 F 1 "331" H 4620 1505 50  0000 L CNN
-F 2 "Resistors_SMD:R_0805_HandSoldering" V 4480 1550 50  0001 C CNN
+F 2 "Resistor_SMD:R_0805_2012Metric_Pad1.15x1.40mm_HandSolder" V 4480 1550 50  0001 C CNN
 F 3 "~" H 4550 1550 50  0001 C CNN
 	1    4550 1550
@@
 F 0 "R5" H 2270 2246 50  0000 L CNN
 F 1 "104" H 2270 2155 50  0000 L CNN
-F 2 "Resistors_SMD:R_0805_HandSoldering" V 2130 2200 50  0001 C CNN
+F 2 "Resistor_SMD:R_0805_2012Metric_Pad1.15x1.40mm_HandSolder" V 2130 2200 50  0001 C CNN
 F 3 "~" H 2200 2200 50  0001 C CNN
 	1    2200 2200
@@
 F 0 "D2" V 2238 1483 50  0000 R CNN
 F 1 "LED" V 2147 1483 50  0000 R CNN
-F 2 "LEDs:LED_0805_HandSoldering" H 2200 1600 50  0001 C CNN
+F 2 "LED_SMD:LED_0805_2012Metric_Castellated" H 2200 1600 50  0001 C CNN
 F 3 "~" H 2200 1600 50  0001 C CNN
 	1    2200 1600

Commit message: update,
Parts:
- R4: value 331 -> 680
Changed lines of the file:
@@
 P 4550 1550
 F 0 "R4" H 4620 1596 50  0000 L CNN
-F 1 "331" H 4620 1505 50  0000 L CNN
+F 1 "680" H 4620 1505 50  0000 L CNN
 F 2 "Resistor_SMD:R_0805_2012Metric_Pad1.15x1.40mm_HandSolder" V 4480 1550 50  0001 C CNN
 F 3 "~" H 4550 1550 50  0001 C CNN

Commit message: update,
Parts:
- added 5V1, GND1, SSR1, SSR2: TestPoint, TestPoint:TestPoint_Loop_D1.80mm_Drill1.0mm_Beaded, symbol Connector:TestPoint
- added C1: 105, Capacitor_SMD:CP_Elec_4x3, symbol Device:C
- added D3: LED, LED_SMD:LED_0805_2012Metric_Castellated, symbol Device:LED
- added Q2: 2N3904, Package_TO_SOT_SMD:TSOT-23_HandSoldering, symbol customized_Transistor_BJT:2N3904
- added R6, R8: 331, Resistor_SMD:R_0805_2012Metric_Pad1.15x1.40mm_HandSolder, symbol Device:R
- added R7: 103, Resistor_SMD:R_0805_2012Metric_Pad1.15x1.40mm_HandSolder, symbol Device:R
- added R9: 680, Resistor_SMD:R_0805_2012Metric_Pad1.15x1.40mm_HandSolder, symbol Device:R
- added U2: OMRON G3MB-202P, footprint-lib:OMRON-G3MB-202P, symbol taobao-components:S108T02
- J1: footprint Connector_PinHeader_2.54mm:PinHeader_1x03_P2.54mm_Vertical -> Connector_PinHeader_2.54mm:PinHeader_1x04_P2.54mm_Vertical; symbol Connector_Generic:Conn_01x03 -> Connector_Generic:Conn_01x04
- J2: value Conn_01x02 -> SSR_OUTPUT; footprint w_conn_mpt:mpt_0,5%2f2-2,54 -> w_conn_mpt:mpt_0,5%2f4-2,54; symbol Connector_Generic:Conn_01x02 -> Connector_Generic:Conn_01x04
Connections:
- net labels added: SSR1_IN1, SSR1_IN2, SSR1_OUT1, SSR1_OUT2, SSR2_IN1, SSR2_IN2, SSR2_OUT1, SSR2_OUT2, SSR_CONTROL1, SSR_CONTROL2
- net labels removed: SIG_CONTROL, SSR_IN1, SSR_IN2, SSR_OUT1, SSR_OUT2
- wire segments 29 -> 63
Other:
- moved on the sheet: D1, D2, Q1, R1, R2, R3, R4, R5, U1

Commit message: update,
Parts:
- Q1: symbol customized_Transistor_BJT:2N3904 -> taobao-transistor:2N3904(1AM)
Connections:
- net GND: now also Q1.2 (E); no longer Q1.1 (E)
- net at R1.1, R2.1: now also Q1.1 (B); no longer Q1.2 (B)
Changed lines of the file:
@@
 $EndComp
 $Comp
-L customized_Transistor_BJT:2N3904 Q1
+L taobao-transistor:2N3904(1AM) Q1
 U 1 1 5BB9F740
 P 9250 2900
